File: Sweep Bling LP/pcb/sweepbling-lp__pcb.kicad_pcb (KiCad board)
At the start: 2 copper layers, 216.9 x 86.9 mm, 59 parts, among them SW1 SW_Push, SW10 SW_Push, SW10_r1 SW_Push, SW11 SW_Push, SW11_r1 SW_Push, SW12 SW_Push, SW12_r1 SW_Push, SW13 SW_Push, SW13_r1 SW_Push, SW14 SW_Push, SW14_r1 SW_Push, SW15 SW_Push, SW15_r1 SW_Push, SW16 SW_Push, SW16_r1 SW_Push, SW17 SW_Push, SW17_r1 SW_Push, SW1_r1 SW_Push, SW2 SW_Push, SW2_r1 SW_Push, SW3 SW_Push, SW3_r1 SW_Push, SW4 SW_Push, SW4_r1 SW_Push, SW5 SW_Push, SW5_r1 SW_Push, SW6 SW_Push, SW6_r1 SW_Push, SW7 SW_Push, SW7_r1 SW_Push, SW8 SW_Push, SW8_r1 SW_Push, SW9 SW_Push, SW9_r1 SW_Push, U1 ProMicro-kbd, U2 ProMicro-kbd

Commit message: made sweep bling LP Choc v2
Parts:
- SW1, SW10, SW10_r1, SW11, SW11_r1, SW12, SW12_r1, SW13, SW13_r1, SW14, SW14_r1, SW15, SW15_r1, SW16, SW16_r1, SW17, SW17_r1, SW1_r1, SW2, SW2_r1, SW3, SW3_r1, SW4, SW4_r1, SW5, SW5_r1, SW6, SW6_r1, SW7, SW7_r1, SW8, SW8_r1, SW9, SW9_r1: footprint * duckyb-collection:SW_Hotswap_Kailh_Choc_V1_tweaked -> PCM_marbastlib-xp-choc:SW_choc_v2_HS_CPG135001S30_1u; moved to B.Cu
Connections:
- SW1 pad 1: Switch1 -> gnd
- SW1 pad 2: gnd -> Switch1
- SW10 pad 1: Switch10 -> gnd
- SW10 pad 2: gnd -> Switch10
- SW10_r1 pad 1: Switch10_r -> gnd_r
- SW10_r1 pad 2: gnd_r -> Switch10_r
- SW11 pad 1: Switch11 -> gnd
- SW11 pad 2: gnd -> Switch11
- SW11_r1 pad 1: Switch11_r -> gnd_r
- SW11_r1 pad 2: gnd_r -> Switch11_r
- SW12 pad 1: Switch12 -> gnd
- SW12 pad 2: gnd -> Switch12
- SW12_r1 pad 1: Switch12_r -> gnd_r
- SW12_r1 pad 2: gnd_r -> Switch12_r
- SW13 pad 1: Switch13 -> gnd
- SW13 pad 2: gnd -> Switch13
- SW13_r1 pad 1: Switch13_r -> gnd_r
- SW13_r1 pad 2: gnd_r -> Switch13_r
- SW14 pad 1: Switch14 -> gnd
- SW14 pad 2: gnd -> Switch14
- SW14_r1 pad 1: Switch14_r -> gnd_r
- SW14_r1 pad 2: gnd_r -> Switch14_r
- SW15 pad 1: Switch15 -> gnd
- SW15 pad 2: gnd -> Switch15
- SW15_r1 pad 1: Switch15_r -> gnd_r
- SW15_r1 pad 2: gnd_r -> Switch15_r
- SW16 pad 1: Switch16 -> gnd
- SW16 pad 2: gnd -> Switch16
- SW16_r1 pad 1: Switch16_r -> gnd_r
- SW16_r1 pad 2: gnd_r -> Switch16_r
- SW17 pad 1: Switch17 -> gnd
- SW17 pad 2: gnd -> Switch17
- SW17_r1 pad 1: Switch17_r -> gnd_r
- SW17_r1 pad 2: gnd_r -> Switch17_r
- SW1_r1 pad 1: Switch1_r -> gnd_r
- SW1_r1 pad 2: gnd_r -> Switch1_r
- SW2 pad 1: Switch2 -> gnd
- SW2 pad 2: gnd -> Switch2
- SW2_r1 pad 1: Switch2_r -> gnd_r
- SW2_r1 pad 2: gnd_r -> Switch2_r
- SW3 pad 1: Switch3 -> gnd
- SW3 pad 2: gnd -> Switch3
- SW3_r1 pad 1: Switch3_r -> gnd_r
- SW3_r1 pad 2: gnd_r -> Switch3_r
- SW4 pad 1: Switch4 -> gnd
- SW4 pad 2: gnd -> Switch4
- SW4_r1 pad 1: Switch4_r -> gnd_r
- SW4_r1 pad 2: gnd_r -> Switch4_r
- SW5 pad 1: Switch5 -> gnd
- SW5 pad 2: gnd -> Switch5
- SW5_r1 pad 1: Switch5_r -> gnd_r
- SW5_r1 pad 2: gnd_r -> Switch5_r
- SW6 pad 1: Switch6 -> gnd
- SW6 pad 2: gnd -> Switch6
- SW6_r1 pad 1: Switch6_r -> gnd_r
- SW6_r1 pad 2: gnd_r -> Switch6_r
- SW7 pad 1: Switch7 -> gnd
- SW7 pad 2: gnd -> Switch7
- SW7_r1 pad 1: Switch7_r -> gnd_r
- SW7_r1 pad 2: gnd_r -> Switch7_r
- SW8 pad 1: Switch8 -> gnd
- SW8 pad 2: gnd -> Switch8
- SW8_r1 pad 1: Switch8_r -> gnd_r
- SW8_r1 pad 2: gnd_r -> Switch8_r
- SW9 pad 1: Switch9 -> gnd
- SW9 pad 2: gnd -> Switch9
- SW9_r1 pad 1: Switch9_r -> gnd_r
- SW9_r1 pad 2: gnd_r -> Switch9_r
Routing:
- net Switch17_r: track 32.4 -> 18.9 mm
- net Switch4_r: track 77.7 -> 70.0 mm
- net Switch3_r: track 96.2 -> 91.1 mm
- net Switch2_r: track 119.9 -> 116.4 mm
- net Switch6: track 105.4 -> 108.6 mm
- net Switch1_r: track 123.6 -> 120.8 mm
- net Switch6_r: track 129.4 -> 131.9 mm
- net Switch17: track 33.8 -> 31.9 mm
- net Switch1: track 136.4 -> 138.2 mm
- net Switch8: track 60.3 -> 61.7 mm
- net Switch11_r: track 101.4 -> 102.8 mm
- net Switch12: track 102.4 -> 103.7 mm
- net Switch7: track 80.7 -> 82.0 mm
- net Switch12_r: track 80.2 -> 81.4 mm
- net Switch18_r: track 47.6 -> 48.8 mm
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